File: CH573_KIT/CH573_KIT.kicad_pcb (KiCad board)
At the start: 2 copper layers, 39.5 x 52.5 mm, 51 parts, among them J1 BAT, J2 2.54 4P, J3 Conn_02x05_Odd_Even, J4 Conn_02x08_Odd_Even, J5 KF2510-4P, J6 Conn_02x05_Odd_Even, J7 KF2510-4P, J8 Conn_02x03_Odd_Even, SW1 SW_Push, SW2 SW_Push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

Commit message: pcb
Parts:
- removed J7: KF2510-4P, Connector_Molex:Molex_KK-254_AE-6410-04A_1x04_P2.54mm_Vertical
- removed J8: Conn_02x03_Odd_Even, Connector_PinHeader_2.54mm:PinHeader_2x03_P2.54mm_Vertical
- C13: footprint Capacitor_SMD:C_0805_2012Metric -> Capacitor_SMD:C_0603_1608Metric
- C15, C16: value 2.2uF 25V -> NC
- J3, J6: value Conn_02x05_Odd_Even -> Conn_02x06_Odd_Even; footprint Connector_PinHeader_2.54mm:PinHeader_2x05_P2.54mm_Vertical -> Connector_PinHeader_2.54mm:PinHeader_2x06_P2.54mm_Vertical
- J5: footprint Connector_Molex:Molex_KK-254_AE-6410-04A_1x04_P2.54mm_Vertical -> Connector_Molex:Molex_PicoBlade_53047-0410_1x04_P1.25mm_Vertical
- moved D3 81.8 mm to (183.0, 60.2), turned to 180 degrees
- moved R2 80.3 mm to (180.0, 60.2)
- moved F2 75.5 mm to (177.8, 68.8), turned to 180 degrees
- moved D5 75.2 mm to (178.0, 62.5), turned to 180 degrees
- moved F1 70.3 mm to (177.0, 60.2), turned to 180 degrees
- moved L2 68.3 mm to (177.8, 65.2)
- moved D6 67.0 mm to (171.0, 63.5), turned to -90 degrees
- moved J1 63.3 mm to (181.5, 54.8), turned to 180 degrees
- moved C13 60.5 mm to (177.8, 67.2), turned to 180 degrees
- moved D1 57.7 mm to (181.5, 58.0)
- moved J5 56.9 mm to (182.1, 63.4), turned to -90 degrees
- moved C7 56.4 mm to (174.0, 61.8), turned to 180 degrees
- moved R4 54.1 mm to (174.0, 60.2), turned to 180 degrees
- moved C15 26.2 mm to (141.5, 73.8)
- moved SW1 26.2 mm to (139.0, 73.8)
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Connections:
- C16 pad 1: /PB23 -> /NRST
- D5 pad 2: Net-(D5-Pad2) -> Net-(C7-Pad1)
- D6 pad 2: Net-(D6-Pad2) -> +3V3
- F1 pad 1: Net-(D5-Pad2) -> Net-(F1-Pad1)
- F2 pad 1: Net-(D6-Pad2) -> Net-(C13-Pad1)
- J3 pad 1: unconnected-(J3-Pad1) -> VDD
- J3 pad 10: unconnected-(J3-Pad10) -> /PB4
- J3 pad 2: unconnected-(J3-Pad2) -> VDD
- J3 pad 3: unconnected-(J3-Pad3) -> /PB15
- J3 pad 4: unconnected-(J3-Pad4) -> /PB14
- J3 pad 5: unconnected-(J3-Pad5) -> /PB13
- J3 pad 6: unconnected-(J3-Pad6) -> /PB12
- J3 pad 7: unconnected-(J3-Pad7) -> /PB11
- J3 pad 8: unconnected-(J3-Pad8) -> /PB10
- J3 pad 9: unconnected-(J3-Pad9) -> /PB7
- J5 pad 2: Net-(D5-Pad2) -> Net-(F1-Pad1)
- J5 pad 3: Net-(D5-Pad2) -> Net-(F1-Pad1)
- J6 pad 1: unconnected-(J6-Pad1) -> GND
- J6 pad 2: unconnected-(J6-Pad2) -> GND
- SW2 pad 1: /PB23 -> /NRST
- U1 pad 16: /PB23 -> /NRST
Routing:
- net /PB15: track 0.00 -> 49.8 mm, vias 0 -> 2
- net VDD: track 3.58 -> 49.0 mm
- net /PB14: track 0.00 -> 43.5 mm
- net VBUS: track 0.00 -> 31.1 mm
- net /VDD_AHT: track 0.00 -> 27.1 mm
- net /AHT_CLK: track 0.00 -> 25.9 mm
- net /AHT_DIO: track 0.00 -> 25.6 mm
- net /NRST: track 0.00 -> 21.5 mm
- net /PB13: track 0.00 -> 18.2 mm
- net /USB1_DP: track 0.00 -> 17.4 mm
- net /PB7: track 0.00 -> 17.2 mm
- net /PB11: track 0.00 -> 16.8 mm
- net /USB1_DN: track 0.00 -> 16.2 mm
- net /CH_TX: track 3.19 -> 18.2 mm
- net /CH_RX: track 3.78 -> 18.4 mm
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- added copper zone on F.Cu, net +5V
- added copper zone on B.Cu, net GND
- added copper zone on F.Cu, net GND
- added copper zone on F.Cu, net Net-(AE1-Pad1)
- added copper zone on F.Cu, net Net-(D2-Pad2)
- added copper zone on F.Cu, net Net-(L2-Pad1)
Other:
- board text added: "V D C G"
