File: CH573_KIT/CH573_KIT.kicad_pcb (KiCad board)
At the start: 2 copper layers, 39.5 x 52.5 mm, 50 parts, among them J1 BAT, J2 2.54 4P, J3 Conn_02x06_Odd_Even, J4 Conn_02x08_Odd_Even, J5 KF2510-4P, J6 Conn_02x06_Odd_Even, SW1 SW_Push, SW2 SW_Push, U1 CH573F, U2 TPS62203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

Commit message: 1.0
Parts:
- added R7: NC, Resistor_SMD:R_0603_1608Metric, B.Cu at (180.0, 64.0)
- D1, D2, D4: value D_Schottky -> MBR0520
- D3: value POWER LED -> GLEEN LED
- D5: value 5.5V -> SMFJ6.0
- D6: value 5.5V -> SMF3.3A
- L2: value 10uH -> NLV25T 10uH
Connections:
- USB1 pad B6: /USB1_DP -> (no net)
- USB1 pad B7: /USB1_DN -> (no net)
- USB2 pad B6: /USB2_DP -> (no net)
- USB2 pad B7: /USB2_DN -> (no net)
Routing:
- net VBUS: track 31.1 -> 33.2 mm
- net Net-(F1-Pad1): track 8.96 -> 11.1 mm
Other:
- board text added: "Short"
