File: CH573_KIT/CH573_KIT.kicad_sch (KiCad schematic)
At the start: 34 parts

Commit message: 初步完成原理图
Parts:
- removed D?: POWER LED, symbol Device:LED
- removed J? (x2): SHORT, symbol Connector:Conn_01x02_Male
- removed J? (x8): PIN, symbol Connector:Conn_01x01_Male
- removed R?: 10k, symbol Device:R
- removed U?: LM3671, Package_TO_SOT_SMD:SOT-23-5, symbol POWER:LM3671
- added D?: POWER LED, symbol Device:LED
- added D? (x2): 5.5V, symbol Device:D_TVS
- added F? (x2): 200mA 6V, symbol Device:Fuse
- added J?: 2.54 4P, symbol Connector:Conn_01x04_Male
- added J? (x2): 2.54 10P, symbol Connector:Conn_01x10_Male
- added J? (x2): KF2510-4P, symbol Connector:Conn_01x04_Male
- added R?: 10k, symbol Device:R
- added U?: LM3671-3.3V, Package_TO_SOT_SMD:SOT-23-5, symbol POWER:LM3671
- C?: value 4.7uF 16V -> 10uF 10V
- J?: value SHORT -> BAT
Connections:
- net +3V3: now also F?.2, J?.1 (Pin_1)
- net GND: now also D?.1 (A1), D?.1 (A1), D?.1 (K), J?.4 (Pin_4), J?.4 (Pin_4), J?.4 (Pin_4), U?.2 (GND)
- net PB14: now also J?.2 (Pin_2)
- net PB15: now also J?.3 (Pin_3)
- net at C?.1, L?.2: now also J?.1 (Pin_1), U?.4 (FB)
- net at C?.1, R?.1: now also F?.2, U?.1 (VIN)
- net VBUS: now reaches D?.1 (K), D?.1 (K)
- net VBUS: now also J?.1 (Pin_1), R?.1
- net at L?.1: now also U?.5 (SW)
- net at R?.2: now also U?.3 (EN)
- new net: D?.2 (A2), F?.1, J?.2 (Pin_2), J?.3 (Pin_3) (x2)
- new net: D?.2 (A), R?.2
Other:
- note added: "1/2 电流测量"
- note added: "3/4 电压测量"
- note added: "DEBUG"
- note added: "电源输入 3.5V MIN 5.5V MAX"
- note removed: "把测试端子做成一个器件"
- note removed: "电源输入短接帽"
- note removed: "电源输出短接帽"
- note removed: "输入电压检测端"
- note removed: "输入电流检测端"
- note removed: "输出电压检测端"
- note removed: "输出电流检测端"
- moved on the sheet: AE?, C?, D?, L?, R?, U?A, U?B, Y?

Commit message: pcb
Parts:
- removed J? (x2): 2.54 10P, symbol Connector:Conn_01x10_Male
- removed R? (x2): 5.1k, symbol Device:R
- removed U?: LM3671-3.3V, Package_TO_SOT_SMD:SOT-23-5, symbol POWER:LM3671
- removed U? (x2): CH573F, Package_DFN_QFN:QFN-28-1EP_4x4mm_P0.4mm_EP2.3x2.3mm, symbol WCH:CH573F
- removed Y?: Crystal, symbol Device:Crystal
- added C10, C12, C9: 1uF 25V, Capacitor_SMD:C_0603_1608Metric, symbol Device:C
- added C11, C14, C8: 10uF 10V, Capacitor_SMD:C_0603_1608Metric, symbol Device:C
- added C15, C16: 100nF 50V, Capacitor_SMD:C_0603_1608Metric, symbol Device:C
- added C2: 10nF 50V, Capacitor_SMD:C_0603_1608Metric, symbol Device:C
- added D4: D_Schottky, Diode_SMD:D_SOD-123, symbol Device:D_Schottky
- added J3, J6: Conn_02x05_Odd_Even, Connector_PinHeader_2.54mm:PinHeader_2x05_P2.54mm_Vertical, symbol Connector_Generic:Conn_02x05_Odd_Even
- added J4: Conn_02x08_Odd_Even, Connector_PinHeader_2.54mm:PinHeader_2x08_P2.54mm_Vertical, symbol Connector_Generic:Conn_02x08_Odd_Even
- added J8: Conn_02x03_Odd_Even, Connector_PinHeader_2.54mm:PinHeader_2x03_P2.54mm_Vertical, symbol Connector_Generic:Conn_02x03_Odd_Even
- added R3: 1M, Resistor_SMD:R_0603_1608Metric, symbol Device:R
- added R5, R6: 4.7k, Resistor_SMD:R_0603_1608Metric, symbol Device:R
- added SW1, SW2: SW_Push, Button_Switch_SMD:SW_SPST_B3U-1000P, symbol Switch:SW_Push
- added U1: CH573F, Package_DFN_QFN:QFN-28-1EP_4x4mm_P0.4mm_EP2.3x2.3mm, symbol NT_WCH:CH573F
- added U2: TPS62203, Package_TO_SOT_SMD:SOT-23-5, symbol NT_POWER:TPS62203
- added U3: XC6206, Package_TO_SOT_SMD:SOT-23, symbol NT_POWER:XC6206
- added U4: CH343P, Package_DFN_QFN:QFN-16-1EP_3x3mm_P0.5mm_EP1.7x1.7mm, symbol NT_WCH:CH343P
- added U5: AHT21, NT_Sensor:AHT21, symbol NT_Sensor:AHT21
- added USB2: USB_C_Plug_USB2.0, Connector_USB:USB_C_Receptacle_HRO_TYPE-C-31-M-12, symbol Connector:USB_C_Plug_USB2.0
- added Y1: Crystal_32MHz, Crystal:Crystal_SMD_2016-4Pin_2.0x1.6mm, symbol Device:Crystal_GND24
- AE1: renamed from AE?; footprint (none) -> NT_RF:CA-C03
- C1, C3, C4, C5, C6, C7: renamed from C?; footprint (none) -> Capacitor_SMD:C_0603_1608Metric
- C13: renamed from C?; footprint (none) -> Capacitor_SMD:C_0805_2012Metric
- D1, D2: renamed from D?; footprint (none) -> Diode_SMD:D_SOD-123
- D3: renamed from D?; footprint (none) -> LED_SMD:LED_0603_1608Metric
- D5, D6: renamed from D?; footprint (none) -> Diode_SMD:D_SOD-123F
- F1, F2: renamed from F?; footprint (none) -> Fuse:Fuse_0603_1608Metric
- J1: renamed from J?; footprint (none) -> Connector_PinHeader_2.54mm:PinHeader_1x02_P2.54mm_Vertical
- J2: renamed from J?; footprint (none) -> Connector_PinHeader_2.54mm:PinHeader_1x04_P2.54mm_Vertical
- J5, J7: renamed from J?; footprint (none) -> Connector_Molex:Molex_KK-254_AE-6410-04A_1x04_P2.54mm_Vertical
- L1: renamed from L?; footprint (none) -> Inductor_SMD:L_TDK_NLV25_2.5x2.0mm
- L2: renamed from L?; value 2.2uH -> 10uH; footprint (none) -> Inductor_SMD:L_TDK_NLV25_2.5x2.0mm
- R1, R2, R4: renamed from R?; footprint (none) -> Resistor_SMD:R_0603_1608Metric
- USB1: renamed from P?; footprint (none) -> Connector_USB:USB_C_Receptacle_HRO_TYPE-C-31-M-12
Connections:
- net +3V3: now also J4.1 (Pin_1); no longer C3.1, J2.1 (Pin_1)
- net BOOT: now also C15.1, SW1.1, U1.17 (PB22/TMR3/RXD2)
- net GND: now also C10.2, C11.2, C12.2, C14.2, C15.2, C16.2, C2.2, C8.2, C9.2, J8.2 (Pin_2), J8.4 (Pin_4), J8.6 (Pin_6), R3.1, SW1.2, SW2.2, U1.29 (GND), U2.2 (GND), U3.1 (VSS), U4.17 (GND), U4.2 (GND), U5.5 (GND), USB2.A1 (GND), USB2.A12 (GND), USB2.B1 (GND), USB2.B12 (GND), Y1.2, Y1.4
- net PA10: now also U1.2 (PA10/X32KI/TMR1)
- net PA11: now also U1.1 (PA11/X32KO/TMR2)
- net PA12: now also U1.28 (PA12/SCS/PWM4/AIN2)
- net PA13: now also U1.27 (PA13/SCK0/PWM5/AIN3)
- net PA14: now also U1.26 (PA14/MOSI/TXD0_/AIN4)
- net PA15: now also U1.25 (PA15/MISO/RXD0_/AIN5)
- net PA4: now also U1.23 (PA4/RXD3/AIN0)
- net PA5: now also U1.24 (PA5/TXD3/AIN1)
- net PB10: now also J4.4 (Pin_4), U1.13 (PB10/UD-/TMR1_); no longer USB1.A7 (D-)
- net PB11: now also J4.6 (Pin_6), U1.12 (PB11/UD+/TMR2_); no longer USB1.A6 (D+)
- net PB12: now also U1.11 (PB12/SCS_/RXD1_)
- net PB13: now also U1.10 (PB13/SCK0_/TXD1_)
- net PB14: now also U1.9 (PB14/TIO/MOSI_/PWM10/DSR)
- net PB15: now also U1.8 (PB15/TCK/MISO_/DTR)
- net PB4: now also U1.15 (PB4/RXD0/PWM7)
- net PB7: now also U1.14 (PB7/TXD0/PWM9)
- net VBUS: now also D4.1 (K)
- net VSW: now also U1.22 (VDCIA), U1.3 (VDCID)
- net X32MI: now also U1.19 (X32MI), Y1.3
- net X32MO: now also U1.18 (X32MO), Y1.1
- net at L1.1: now also U1.4 (VSW)
- net at C4.1: now also U1.20 (VINTA)
- net at L2.1: now also U2.5 (SW)
- net at C13.1, J7.1 (Pin_1), L2.2: now also U2.4 (FB)
- net at C7.1, F1.2, R4.1: now also U2.1 (VIN)
- net at R4.2: now also U2.3 (EN)
- net at AE1.1 (A): now also U1.21 (ANT)
- net CC1: no longer names the net of USB1.A5 (CC)
- net CC2: no longer names the net of USB1.B5 (VCONN)
- new net: C2.1, R3.2, USB2.S1 (SHIELD)
- new net +3.3V_UART: C10.1, C11.1, C12.1, C9.1, U3.2 (Vout), U4.1 (VIO), U4.3 (VDD5), U4.6 (V3)
- new net +5V: C8.1, D4.2 (A), U3.3 (VCC), U4.9 (VBUS), USB2.A4 (VBUS), USB2.A9 (VBUS), USB2.B4 (VBUS), USB2.B9 (VBUS)
- new net AHT_CLK: J4.13 (Pin_13), R6.2, U5.3 (SCL)
- new net AHT_DIO: J4.11 (Pin_11), R5.2, U5.4 (SDA)
- new net CH_RX: J4.8 (Pin_8), U1.6 (PA8/RXD1/AIN12)
- new net CH_TX: J4.10 (Pin_10), U1.7 (PA9/TMR0/TXD1/AIN13)
- new net I2C_CK: J4.14 (Pin_14)
- new net I2C_IO: J4.12 (Pin_12)
- new net NRST: C16.1, SW2.1, U1.16 (PB23/RST#/TMR0_/TXD2/PWM11)
- new net USB1_DN: J4.3 (Pin_3), USB1.A7 (D-)
- new net USB1_DP: J4.5 (Pin_5), USB1.A6 (D+)
- new net USB2_DN: U4.8 (UD-), USB2.A7 (D-)
- new net USB2_DP: U4.7 (UD+), USB2.A6 (D+)
- new net USB_RX: J4.9 (Pin_9), U4.5 (RXD)
- new net USB_TX: J4.7 (Pin_7), U4.4 (TXD)
- new net VDD: C3.1, J2.1 (Pin_1), J4.16 (Pin_16), J4.2 (Pin_2), J8.1 (Pin_1), J8.3 (Pin_3), J8.5 (Pin_5), U1.5 (VIO33/VDD33)
- new net VDD_AHT: C14.1, J4.15 (Pin_15), R5.1, R6.1, U5.2 (VCC)
- no-connect marks 0 -> 11
Other:
- note added: "H/D USB"
- note added: "串口 USB"
- note added: "直流电源输入 3.5V MIN 5.5V MAX"
- note removed: "USB输入"
- note removed: "电源稳压电路"
- note removed: "电源输入 3.5V MIN 5.5V MAX"
- note removed: "锂电池/可调电源输入"
- moved on the sheet: AE1, C1, C13, C3, C4, C5, C6, C7, D1, D2, D3, D5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

Commit message: pcb
Parts:
- removed J3, J6: Conn_02x05_Odd_Even, Connector_PinHeader_2.54mm:PinHeader_2x05_P2.54mm_Vertical, symbol Connector_Generic:Conn_02x05_Odd_Even
- removed J7: KF2510-4P, Connector_Molex:Molex_KK-254_AE-6410-04A_1x04_P2.54mm_Vertical, symbol Connector:Conn_01x04_Male
- removed J8: Conn_02x03_Odd_Even, Connector_PinHeader_2.54mm:PinHeader_2x03_P2.54mm_Vertical, symbol Connector_Generic:Conn_02x03_Odd_Even
- added J3, J6: Conn_02x06_Odd_Even, Connector_PinHeader_2.54mm:PinHeader_2x06_P2.54mm_Vertical, symbol Connector_Generic:Conn_02x06_Odd_Even
- C13: footprint Capacitor_SMD:C_0805_2012Metric -> Capacitor_SMD:C_0603_1608Metric
- C15, C16: value 100nF 50V -> NC
- J5: footprint Connector_Molex:Molex_KK-254_AE-6410-04A_1x04_P2.54mm_Vertical -> Connector_Molex:Molex_PicoBlade_53047-0410_1x04_P1.25mm_Vertical
Connections:
- net +3V3: now also D6.2 (A2)
- net BOOT: now also J3.12 (Pin_12)
- net GND: now also J6.1 (Pin_1), J6.2 (Pin_2)
- net NRST: now also J3.11 (Pin_11)
- net PB10: now also J3.8 (Pin_8)
- net PB11: now also J3.7 (Pin_7)
- net PB12: now also J3.6 (Pin_6)
- net PB13: now also J3.5 (Pin_5)
- net PB14: now also J3.4 (Pin_4)
- net PB15: now also J3.3 (Pin_3)
- net PB4: now also J3.10 (Pin_10)
- net PB7: now also J3.9 (Pin_9)
- net VDD: now also J3.1 (Pin_1), J3.2 (Pin_2)
- net at C7.1, F1.2, R4.1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: now also D5.2 (A2)
- net at C13.1, L2.2, U2.4 (FB): now also F2.1
- net at F1.1, J5.2 (Pin_2), J5.3 (Pin_3): no longer D5.2 (A2)
Other:
- note added: "(100nF 50V)"
- moved on the sheet: C1, C13, C14, C15, C2, C7, D1, D2, D3, D4, D5, D6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

Commit message: V1.0
Parts:
- SW1, SW2: footprint Button_Switch_SMD:SW_SPST_B3U-1000P -> NT_Switch:SW_Che_2x4x3.5
Connections:
- net PB12 is gone; now on net I2C_IO: J3.6 (Pin_6), U1.11 (PB12/SCS_/RXD1_)
- net PB13 is gone; now on net I2C_CK: J3.5 (Pin_5), U1.10 (PB13/SCK0_/TXD1_)
- net CH_RX: now also J6.4 (Pin_4)
- net CH_TX: now also J6.3 (Pin_3)
- net PA10: now also J6.6 (Pin_6)
- net PA11: now also J6.5 (Pin_5)
- net PA12: now also J6.8 (Pin_8)
- net PA13: now also J6.7 (Pin_7)
- net PA14: now also J6.10 (Pin_10)
- net PA15: now also J6.9 (Pin_9)
- net PA4: now also J6.11 (Pin_11)
- net PA5: now also J6.12 (Pin_12)
Changed lines of the file:
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@@
-    (stroke (width 0) (type default) (color 0 0 0 0))
-  )
-  (wire (pts (xy 31.75 134.62) (xy 38.1 134.62))
     (stroke (width 0) (type default) (color 0 0 0 0))
   )
@@
   )
   (wire (pts (xy 22.86 127) (xy 38.1 127))
-    (stroke (width 0) (type default) (color 0 0 0 0))
-  )
-  (wire (pts (xy 31.75 137.16) (xy 38.1 137.16))
     (stroke (width 0) (type default) (color 0 0 0 0))
   )
@@
     (stroke (width 0) (type default) (color 0 0 0 0))
   )
+  (wire (pts (xy 22.86 137.16) (xy 38.1 137.16))
+    (stroke (width 0) (type default) (color 0 0 0 0))
+  )
   (wire (pts (xy 162.56 73.66) (xy 170.18 73.66))
     (stroke (width 0) (type default) (color 0 0 0 0))
@@
     (stroke (width 0) (type default) (color 0 0 0 0))
   )
+  (wire (pts (xy 22.86 134.62) (xy 38.1 134.62))
+    (stroke (width 0) (type default) (color 0 0 0 0))
+  )
   (wire (pts (xy 97.79 132.08) (xy 105.41 132.08))
     (stroke (width 0) (type default) (color 0 0 0 0))
@@
     (effects (font (size 1.27 1.27)) (justify left bottom))
   )
+  (label "I2C_CK" (at 22.86 134.62 0)
+    (effects (font (size 1.27 1.27)) (justify left bottom))
+  )
   (label "PB22" (at 148.59 128.27 0)
     (effects (font (size 1.27 1.27)) (justify left bottom))
@@
     (effects (font (size 1.27 1.27)) (justify left bottom))
   )
+  (label "PA9" (at 128.27 140.97 0)
+    (effects (font (size 1.27 1.27)) (justify left bottom))
+  )
   (label "PB11" (at 128.27 123.19 0)
     (effects (font (size 1.27 1.27)) (justify left bottom))
@@
     (effects (font (size 1.27 1.27)) (justify left bottom))
   )
+  (label "PA8" (at 148.59 140.97 0)
+    (effects (font (size 1.27 1.27)) (justify left bottom))
+  )
   (label "CH_RX" (at 22.86 124.46 0)
     (effects (font (size 1.27 1.27)) (justify left bottom))
   )
+  (label "PA4" (at 128.27 151.13 0)
+    (effects (font (size 1.27 1.27)) (justify left bottom))
+  )
   (label "USB2_DN" (at 116.84 54.61 0)
     (effects (font (size 1.27 1.27)) (justify left bottom))
@@
     (effects (font (size 1.27 1.27)) (justify left bottom))
   )
+  (label "PA13" (at 128.27 146.05 0)
+    (effects (font (size 1.27 1.27)) (justify left bottom))
+  )
   (label "AHT_CLK" (at 140.97 88.9 0)
     (effects (font (size 1.27 1.27)) (justify left bottom))
@@
     (effects (font (size 1.27 1.27)) (justify left bottom))
   )
+  (label "PA15" (at 128.27 148.59 0)
+    (effects (font (size 1.27 1.27)) (justify left bottom))
+  )
   (label "VDD_AHT" (at 223.52 73.66 0)
     (effects (font (size 1.27 1.27)) (justify left bottom))
@@
     (effects (font (size 1.27 1.27)) (justify left bottom))
   )
+  (label "PA12" (at 148.59 146.05 0)
+    (effects (font (size 1.27 1.27)) (justify left bottom))
+  )
+  (label "PA10" (at 148.59 143.51 0)
+    (effects (font (size 1.27 1.27)) (justify left bottom))
+  )
   (label "PB23" (at 99.06 137.16 0)
     (effects (font (size 1.27 1.27)) (justify left bottom))
@@
     (effects (font (size 1.27 1.27)) (justify left bottom))
   )
+  (label "I2C_IO" (at 22.86 137.16 0)
+    (effects (font (size 1.27 1.27)) (justify left bottom))
+  )
   (label "PB10" (at 31.75 142.24 0)
     (effects (font (size 1.27 1.27)) (justify left bottom))
@@
     (effects (font (size 1.27 1.27)) (justify left bottom))
   )
+  (label "PA11" (at 128.27 143.51 0)
+    (effects (font (size 1.27 1.27)) (justify left bottom))
+  )
   (label "USB1_DP" (at 140.97 78.74 0)
     (effects (font (size 1.27 1.27)) (justify left bottom))
@@
     (effects (font (size 1.27 1.27)) (justify left bottom))
   )
+  (label "PA5" (at 148.59 151.13 0)
+    (effects (font (size 1.27 1.27)) (justify left bottom))
+  )
   (label "CH_TX" (at 163.83 83.82 0)
     (effects (font (size 1.27 1.27)) (justify left bottom))
@@
   )
   (label "PB22" (at 99.06 134.62 0)
+    (effects (font (size 1.27 1.27)) (justify left bottom))
+  )
+  (label "PA14" (at 148.59 148.59 0)
     (effects (font (size 1.27 1.27)) (justify left bottom))
   )
@@
     (property "Reference" "SW2" (id 0) (at 153.67 176.53 0))
     (property "Value" "SW_Push" (id 1) (at 153.67 179.07 0))
-    (property "Footprint" "Button_Switch_SMD:SW_SPST_B3U-1000P" (id 2) (at 153.67 179.07 0)
+    (property "Footprint" "NT_Switch:SW_Che_2x4x3.5" (id 2) (at 153.67 179.07 0)
       (effects (font (size 1.27 1.27)) hide)
     )
@@
     (pin "1")
   )
-  (symbol (lib_id "Switch:SW_Push") (at 153.67 165.1 0) (unit 1)
+  (symbol (lib_name "SW_Push_1") (lib_id "Switch:SW_Push") (at 153.67 165.1 0) (unit 1)
     (in_bom yes) (on_board yes)
     (property "Reference" "SW1" (id 0) (at 153.67 157.48 0))
     (property "Value" "SW_Push" (id 1) (at 153.67 160.02 0))
-    (property "Footprint" "Button_Switch_SMD:SW_SPST_B3U-1000P" (id 2) (at 153.67 160.02 0)
+    (property "Footprint" "NT_Switch:SW_Che_2x4x3.5" (id 2) (at 153.67 160.02 0)
       (effects (font (size 1.27 1.27)) hide)
     )
@@
     )
     (path "/aed7eb4d-03e5-4d1a-91ed-ac61b1481335"
-      (reference "SW1") (unit 1) (value "SW_Push") (footprint "Button_Switch_SMD:SW_SPST_B3U-1000P")
+      (reference "SW1") (unit 1) (value "SW_Push") (footprint "NT_Switch:SW_Che_2x4x3.5")
     )
     (path "/70bcbe16-9d0c-4ddf-9882-4198fc5f0825"
-      (reference "SW2") (unit 1) (value "SW_Push") (footprint "Button_Switch_SMD:SW_SPST_B3U-1000P")
+      (reference "SW2") (unit 1) (value "SW_Push") (footprint "NT_Switch:SW_Che_2x4x3.5")
     )
     (path "/20f9d538-4b5d-48bb-9ceb-3e384d020827"
