File: CH573_KIT/CH573_KIT.kicad_sch (KiCad schematic)
At the start: 49 parts, among them J1 BAT, J2 2.54 4P, J3 Conn_02x06_Odd_Even, J4 Conn_02x08_Odd_Even, J5 KF2510-4P, J6 Conn_02x06_Odd_Even, SW1 SW_Push, SW2 SW_Push, U1 CH573F, U2 TPS62203, U3 XC6206, U4 CH343P, U5 AHT21, Y1 Crystal_32MHz

Commit message: 1.0
Parts:
- added R7: NC, Resistor_SMD:R_0603_1608Metric, symbol Device:R
- C5: value 0.1uF 50V -> 100nF 50V
- D1, D2, D4: value D_Schottky -> MBR0520
- D3: value POWER LED -> GLEEN LED
- D5: value 5.5V -> SMFJ6.0
- D6: value 5.5V -> SMF3.3A
- L2: value 10uH -> NLV25T 10uH
Connections:
- net VBUS: now also R7.2
- net at F1.1, J5.2 (Pin_2), J5.3 (Pin_3): now also R7.1
Other:
- note added: "(0R)"
Changed lines of the file:
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@@
 (kicad_sch (version 20211123) (generator eeschema)
   (paper "A4")
+  (junction (at 152.4 41.91) (diameter 0) (color 0 0 0 0)
+  )
   (junction (at 247.65 41.91) (diameter 0) (color 0 0 0 0)
   )
@@
   )
   (junction (at 93.98 91.44) (diameter 0) (color 0 0 0 0)
+  )
+  (junction (at 154.94 41.91) (diameter 0) (color 0 0 0 0)
   )
   (junction (at 147.32 184.15) (diameter 0) (color 0 0 0 0)
@@
     (stroke (width 0) (type default) (color 0 0 0 0))
   )
-  (wire (pts (xy 160.02 39.37) (xy 160.02 43.18))
+  (wire (pts (xy 160.02 39.37) (xy 160.02 44.45))
     (stroke (width 0) (type default) (color 0 0 0 0))
   )
@@
     (stroke (width 0) (type default) (color 0 0 0 0))
   )
+  (wire (pts (xy 152.4 50.8) (xy 152.4 52.07))
+    (stroke (width 0) (type default) (color 0 0 0 0))
+  )
   (wire (pts (xy 154.94 39.37) (xy 154.94 41.91))
+    (stroke (width 0) (type default) (color 0 0 0 0))
+  )
+  (wire (pts (xy 154.94 41.91) (xy 154.94 52.07))
     (stroke (width 0) (type default) (color 0 0 0 0))
   )
@@
     (stroke (width 0) (type default) (color 0 0 0 0))
   )
+  (wire (pts (xy 152.4 52.07) (xy 154.94 52.07))
+    (stroke (width 0) (type default) (color 0 0 0 0))
+  )
   (wire (pts (xy 220.98 76.2) (xy 219.71 76.2))
     (stroke (width 0) (type default) (color 0 0 0 0))
@@
     (stroke (width 0) (type default) (color 0 0 0 0))
   )
+  (wire (pts (xy 152.4 41.91) (xy 152.4 43.18))
+    (stroke (width 0) (type default) (color 0 0 0 0))
+  )
   (wire (pts (xy 229.87 41.91) (xy 234.95 41.91))
     (stroke (width 0) (type default) (color 0 0 0 0))
@@
     (effects (font (size 1.27 1.27)) (justify left bottom))
   )
-  (text "3/4 电压测量" (at 143.51 48.26 0)
+  (text "3/4 电压测量" (at 149.86 25.4 0)
+    (effects (font (size 1.27 1.27)) (justify left bottom))
+  )
+  (text "(0R)" (at 146.05 52.07 0)
     (effects (font (size 1.27 1.27)) (justify left bottom))
   )
@@
     (effects (font (size 1.27 1.27)) (justify left bottom))
   )
-  (text "1/2 电流测量" (at 143.51 45.72 0)
+  (text "1/2 电流测量" (at 149.86 22.86 0)
     (effects (font (size 1.27 1.27)) (justify left bottom))
   )
@@
       (effects (font (size 1.27 1.27)) (justify left))
     )
-    (property "Value" "0.1uF 50V" (id 1) (at 104.14 184.15 0)
+    (property "Value" "100nF 50V" (id 1) (at 104.14 184.15 0)
       (effects (font (size 1.27 1.27)) (justify left))
     )
@@
     (in_bom yes) (on_board yes) (fields_autoplaced)
     (property "Reference" "D1" (id 0) (at 65.0875 19.05 0))
-    (property "Value" "D_Schottky" (id 1) (at 65.0875 21.59 0))
+    (property "Value" "MBR0520" (id 1) (at 65.0875 21.59 0))
     (property "Footprint" "Diode_SMD:D_SOD-123" (id 2) (at 64.77 25.4 0)
       (effects (font (size 1.27 1.27)) hide)
@@
       (effects (font (size 1.27 1.27)) (justify left))
     )
-    (property "Value" "POWER LED" (id 1) (at 95.25 21.59 0)
+    (property "Value" "GLEEN LED" (id 1) (at 95.25 21.59 0)
       (effects (font (size 1.27 1.27)) (justify left))
     )
@@
     (in_bom yes) (on_board yes)
     (property "Reference" "L2" (id 0) (at 223.52 36.83 90))
-    (property "Value" "10uH" (id 1) (at 224.79 39.37 90))
+    (property "Value" "NLV25T 10uH" (id 1) (at 227.33 39.37 90))
     (property "Footprint" "Inductor_SMD:L_TDK_NLV25_2.5x2.0mm" (id 2) (at 224.79 41.91 0)
       (effects (font (size 1.27 1.27)) hide)
@@
     (in_bom yes) (on_board yes) (fields_autoplaced)
     (property "Reference" "D2" (id 0) (at 65.0875 34.29 0))
-    (property "Value" "D_Schottky" (id 1) (at 65.0875 36.83 0))
+    (property "Value" "MBR0520" (id 1) (at 65.0875 36.83 0))
     (property "Footprint" "Diode_SMD:D_SOD-123" (id 2) (at 64.77 40.64 0)
       (effects (font (size 1.27 1.27)) hide)
@@
     (in_bom yes) (on_board yes) (fields_autoplaced)
     (property "Reference" "D4" (id 0) (at 128.5875 35.56 0))
-    (property "Value" "D_Schottky" (id 1) (at 128.5875 38.1 0))
+    (property "Value" "MBR0520" (id 1) (at 128.5875 38.1 0))
     (property "Footprint" "Diode_SMD:D_SOD-123" (id 2) (at 128.27 41.91 0)
       (effects (font (size 1.27 1.27)) hide)
@@
     )
     (property "Datasheet" "~" (id 3) (at 219.71 149.86 0)
+      (effects (font (size 1.27 1.27)) hide)
+    )
+    (pin "1")
+    (pin "2")
+  )
+  (symbol (lib_id "Device:R") (at 152.4 46.99 180) (unit 1)
+    (in_bom yes) (on_board yes)
+    (property "Reference" "R7" (id 0) (at 148.59 45.72 0))
+    (property "Value" "NC" (id 1) (at 148.59 48.26 0))
+    (property "Footprint" "Resistor_SMD:R_0603_1608Metric" (id 2) (at 154.178 46.99 90)
+      (effects (font (size 1.27 1.27)) hide)
+    )
+    (property "Datasheet" "~" (id 3) (at 152.4 46.99 0)
       (effects (font (size 1.27 1.27)) hide)
     )
@@
     (pin "2")
   )
-  (symbol (lib_id "power:GND") (at 160.02 43.18 0) (unit 1)
-    (in_bom yes) (on_board yes)
-    (property "Reference" "#PWR020" (id 0) (at 160.02 49.53 0)
+  (symbol (lib_id "power:GND") (at 160.02 44.45 0) (unit 1)
+    (in_bom yes) (on_board yes)
+    (property "Reference" "#PWR020" (id 0) (at 160.02 50.8 0)
       (effects (font (size 1.27 1.27)) hide)
     )
     (property "Value" "GND" (id 1) (at 160.02 48.26 0))
-    (property "Footprint" "" (id 2) (at 160.02 43.18 0)
-      (effects (font (size 1.27 1.27)) hide)
-    )
-    (property "Datasheet" "" (id 3) (at 160.02 43.18 0)
+    (property "Footprint" "" (id 2) (at 160.02 44.45 0)
+      (effects (font (size 1.27 1.27)) hide)
+    )
+    (property "Datasheet" "" (id 3) (at 160.02 44.45 0)
       (effects (font (size 1.27 1.27)) hide)
     )
@@
       (effects (font (size 1.27 1.27)) (justify right))
     )
-    (property "Value" "5.5V" (id 1) (at 250.19 48.26 90)
+    (property "Value" "SMF3.3A" (id 1) (at 250.19 48.26 90)
       (effects (font (size 1.27 1.27)) (justify right))
     )
@@
   )
   (symbol (lib_id "Device:D_TVS") (at 172.72 46.99 90) (unit 1)
-    (in_bom yes) (on_board yes) (fields_autoplaced)
-    (property "Reference" "D5" (id 0) (at 175.26 45.7199 90)
+    (in_bom yes) (on_board yes)
+    (property "Reference" "D5" (id 0) (at 173.99 48.26 90)
       (effects (font (size 1.27 1.27)) (justify right))
     )
-    (property "Value" "5.5V" (id 1) (at 175.26 48.2599 90)
+    (property "Value" "SMFJ6.0" (id 1) (at 168.91 50.8 90)
       (effects (font (size 1.27 1.27)) (justify right))
     )
@@
     )
     (path "/3c811405-f5e1-448d-b8b8-eef19b0ae5a8"
-      (reference "C5") (unit 1) (value "0.1uF 50V") (footprint "Capacitor_SMD:C_0603_1608Metric")
+      (reference "C5") (unit 1) (value "100nF 50V") (footprint "Capacitor_SMD:C_0603_1608Metric")
     )
     (path "/7732351b-c136-4fd0-a0be-917db18cb759"
@@
     )
     (path "/54ada65e-b3cc-4a36-9027-e7f804792a60"
-      (reference "D1") (unit 1) (value "D_Schottky") (footprint "Diode_SMD:D_SOD-123")
+      (reference "D1") (unit 1) (value "MBR0520") (footprint "Diode_SMD:D_SOD-123")
     )
     (path "/8272c4bb-82ad-4654-b089-f628a197cd9a"
-      (reference "D2") (unit 1) (value "D_Schottky") (footprint "Diode_SMD:D_SOD-123")
+      (reference "D2") (unit 1) (value "MBR0520") (footprint "Diode_SMD:D_SOD-123")
     )
     (path "/6dc68749-b967-4266-be0d-056867c1be87"
-      (reference "D3") (unit 1) (value "POWER LED") (footprint "LED_SMD:LED_0603_1608Metric")
+      (reference "D3") (unit 1) (value "GLEEN LED") (footprint "LED_SMD:LED_0603_1608Metric")
     )
     (path "/b6e1fe8b-3ebb-4cb8-b869-32345d688843"
-      (reference "D4") (unit 1) (value "D_Schottky") (footprint "Diode_SMD:D_SOD-123")
+      (reference "D4") (unit 1) (value "MBR0520") (footprint "Diode_SMD:D_SOD-123")
     )
     (path "/f884d88b-b792-41cd-9203-0ee6c7f11dab"
-      (reference "D5") (unit 1) (value "5.5V") (footprint "Diode_SMD:D_SOD-123F")
+      (reference "D5") (unit 1) (value "SMFJ6.0") (footprint "Diode_SMD:D_SOD-123F")
     )
     (path "/ec2a6e1f-9d42-4629-8882-f087943c699b"
-      (reference "D6") (unit 1) (value "5.5V") (footprint "Diode_SMD:D_SOD-123F")
+      (reference "D6") (unit 1) (value "SMF3.3A") (footprint "Diode_SMD:D_SOD-123F")
     )
     (path "/a59c9058-54ba-4989-9d0c-d01a7df7cfa9"
@@
     )
     (path "/764acd62-e6f0-401e-9f1a-68faca9ad2e4"
-      (reference "L2") (unit 1) (value "10uH") (footprint "Inductor_SMD:L_TDK_NLV25_2.5x2.0mm")
+      (reference "L2") (unit 1) (value "NLV25T 10uH") (footprint "Inductor_SMD:L_TDK_NLV25_2.5x2.0mm")
     )
     (path "/84d7e0b3-6105-406f-bcfe-0f01b74f2dc6"
@@
       (reference "R6") (unit 1) (value "4.7k") (footprint "Resistor_SMD:R_0603_1608Metric")
     )
+    (path "/d1d5a8e9-87ae-4668-899b-866659896157"
+      (reference "R7") (unit 1) (value "NC") (footprint "Resistor_SMD:R_0603_1608Metric")
+    )
     (path "/aed7eb4d-03e5-4d1a-91ed-ac61b1481335"

Commit message: 1.0
Other:
- note added: "(or 100nF 50V)"
- note removed: "(100nF 50V)"
Changed lines of the file:
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@@
-    (effects (font (size 1.27 1.27)) (justify left bottom))
-  )
-  (text "(100nF 50V)" (at 156.21 172.72 0)
     (effects (font (size 1.27 1.27)) (justify left bottom))
   )
@@
     (effects (font (size 1.27 1.27)) (justify left bottom))
   )
-  (text "(100nF 50V)" (at 156.21 191.77 0)
+  (text "(or 100nF 50V)" (at 156.21 191.77 0)
     (effects (font (size 1.27 1.27)) (justify left bottom))
   )
